Commit message: multi tb3 simulation

File: src/robot_description/urdf/turtlebot3_burger/gz_control.xacro (robot description, xacro)
@@ -1,10 +1,9 @@
 <?xml version="1.0"?>
 <robot xmlns:xacro="http://www.ros.org/wiki/xacro">
-  <xacro:macro name="tb3_gz_control" params="">
+  <xacro:macro name="tb3_gz_control" params="model_name">
     <gazebo>
       <plugin
         filename="libignition-gazebo-diff-drive-system.so"
         name="ignition::gazebo::systems::DiffDrive">
-        <!-- Must match ign model -j exactly -->
         <left_joint>wheel_left_joint</left_joint>
         <right_joint>wheel_right_joint</right_joint>
@@ -12,9 +11,8 @@
         <wheel_radius>0.033</wheel_radius>
         <max_linear_acceleration>0.33</max_linear_acceleration>
-        <!-- Ignition topic (you confirmed /cmd_vel exists) -->
-        <topic>cmd_vel</topic>
+        <topic>/model/${model_name}/cmd_vel</topic>
         <frame_id>odom</frame_id>
         <child_frame_id>base_link</child_frame_id>
-        <odom_topic>odom</odom_topic>
+        <odom_topic>/model/${model_name}/odom</odom_topic>
         <odom_publisher_frequency>30</odom_publisher_frequency>
         <tf_topic>/tf</tf_topic>
@@ -23,5 +21,5 @@
         filename="libignition-gazebo-joint-state-publisher-system.so"
         name="ignition::gazebo::systems::JointStatePublisher">
-        <topic>joint_states</topic>
+        <topic>/model/${model_name}/joint_states</topic>
       </plugin>
     </gazebo>

File: src/robot_description/urdf/turtlebot3_burger/robot.urdf.xacro (robot description, xacro)
@@ -4,6 +4,5 @@
     <color rgba="0.3 0.3 0.3 1.0"/>
   </material>
-  <xacro:arg name="namespace" default="tb3"/>
-  <xacro:arg name="use_sim_time" default="true"/>
+  <xacro:arg name="model_name" default="tb3"/>
   <xacro:include filename="robot_core.xacro" />
   <xacro:include filename="robot_sensors.xacro" />
@@ -11,6 +10,6 @@
   <xacro:macro name="tb3_robot" params="">
     <xacro:tb3_core/>
-    <xacro:tb3_sensors/>
-    <xacro:tb3_gz_control/>
+    <xacro:tb3_sensors model_name="$(arg model_name)"/>
+    <xacro:tb3_gz_control model_name="$(arg model_name)"/>
   </xacro:macro>
   <xacro:tb3_robot/>

File: src/robot_description/urdf/turtlebot3_burger/robot_sensors.xacro (robot description, xacro)
@@ -1,5 +1,5 @@
 <?xml version="1.0"?>
 <robot xmlns:xacro="http://www.ros.org/wiki/xacro">
-  <xacro:macro name="tb3_sensors" params="">
+  <xacro:macro name="tb3_sensors" params="model_name">
     <!-- Laser -->
     <link name="base_scan">
@@ -33,5 +33,5 @@
     <gazebo reference="base_scan">
       <!-- <material>Gazebo/Black</material> -->
-      <sensor name="lds_sensor" type="ray">
+      <sensor name="lds_sensor" type="gpu_lidar">
         <pose>0 0 0 0 0 0</pose>
         <always_on>1</always_on>
@@ -56,6 +56,6 @@
           </noise>
         </lidar>
-        <topic>scan</topic>
-        <gz_frame_id>base_scan</gz_frame_id>
+        <topic>/model/${model_name}/scan</topic>
+        <gz_frame_id>${model_name}/base_scan</gz_frame_id>
       </sensor>
     </gazebo>
@@ -79,6 +79,6 @@
       <always_on>1</always_on>
       <update_rate>200</update_rate>
-      <topic>/imu</topic>
-      <gz_frame_id>$imu_link</gz_frame_id>
+      <topic>/model/${model_name}/imu</topic>
+      <gz_frame_id>${model_name}/imu_link</gz_frame_id>
     </sensor>
   </gazebo>
