Commit message: implement robot config

File: src/cares_simulation/urdf/turtlebot3/robot_core.xacro (robot description, xacro)
@@ -17,5 +17,5 @@
         <origin xyz="-0.032 0 0.0" rpy="0 0 0"/>
         <geometry>
-          <mesh filename="package://robot_description/models/turtlebot3_common/meshes/burger_base.dae"
+          <mesh filename="package://cares_simulation/models/turtlebot3_common/meshes/burger_base.dae"
                 scale="0.001 0.001 0.001"/>
         </geometry>
@@ -47,5 +47,5 @@
           <origin xyz="0 0 0" rpy="${M_PI/2} 0 0"/>
           <geometry>
-            <mesh filename="package://robot_description/models/turtlebot3_common/meshes/tire.dae"
+            <mesh filename="package://cares_simulation/models/turtlebot3_common/meshes/tire.dae"
                   scale="0.001 0.001 0.001"/>
           </geometry>

File: src/cares_simulation/urdf/turtlebot3/robot_sensors.xacro (robot description, xacro)
@@ -7,5 +7,5 @@
         <origin xyz="-0.032 0 0.0" rpy="0 0 0"/>
         <geometry>
-          <mesh filename="package://robot_description/models/turtlebot3_common/meshes/lds.dae"
+          <mesh filename="package://cares_simulation/models/turtlebot3_common/meshes/lds.dae"
                 scale="0.001 0.001 0.001"/>
         </geometry>

Commit message: jethexa urdf

File: src/cares_simulation/urdf/turtlebot3/robot_core.xacro (robot description, xacro)
@@ -17,5 +17,5 @@
         <origin xyz="-0.032 0 0.0" rpy="0 0 0"/>
         <geometry>
-          <mesh filename="package://cares_simulation/models/turtlebot3_common/meshes/burger_base.dae"
+          <mesh filename="package://cares_simulation/models/turtlebot3/burger_base.dae"
                 scale="0.001 0.001 0.001"/>
         </geometry>
@@ -47,5 +47,5 @@
           <origin xyz="0 0 0" rpy="${M_PI/2} 0 0"/>
           <geometry>
-            <mesh filename="package://cares_simulation/models/turtlebot3_common/meshes/tire.dae"
+            <mesh filename="package://cares_simulation/models/turtlebot3/tire.dae"
                   scale="0.001 0.001 0.001"/>
           </geometry>

File: src/cares_simulation/urdf/turtlebot3/robot_sensors.xacro (robot description, xacro)
@@ -7,5 +7,5 @@
         <origin xyz="-0.032 0 0.0" rpy="0 0 0"/>
         <geometry>
-          <mesh filename="package://cares_simulation/models/turtlebot3_common/meshes/lds.dae"
+          <mesh filename="package://cares_simulation/models/turtlebot3/lds.dae"
                 scale="0.001 0.001 0.001"/>
         </geometry>
