Commit message: jethexa urdf

File: src/chroma_simulation/urdf/turtlebot3/robot_core.xacro (robot description, xacro)
@@ -17,5 +17,9 @@
         <origin xyz="-0.032 0 0.0" rpy="0 0 0"/>
         <geometry>
+<<<<<<< HEAD:src/chroma_simulation/urdf/turtlebot3/robot_core.xacro
           <mesh filename="package://chroma_simulation/models/turtlebot3/burger_base.dae"
+=======
+          <mesh filename="package://cares_simulation/models/turtlebot3/burger_base.dae"
+>>>>>>> b0b80ff (jethexa urdf):src/cares_simulation/urdf/turtlebot3/robot_core.xacro
                 scale="0.001 0.001 0.001"/>
         </geometry>
@@ -47,5 +51,9 @@
           <origin xyz="0 0 0" rpy="${M_PI/2} 0 0"/>
           <geometry>
+<<<<<<< HEAD:src/chroma_simulation/urdf/turtlebot3/robot_core.xacro
             <mesh filename="package://chroma_simulation/models/turtlebot3/tire.dae"
+=======
+            <mesh filename="package://cares_simulation/models/turtlebot3/tire.dae"
+>>>>>>> b0b80ff (jethexa urdf):src/cares_simulation/urdf/turtlebot3/robot_core.xacro
                   scale="0.001 0.001 0.001"/>
           </geometry>

File: src/chroma_simulation/urdf/turtlebot3/robot_sensors.xacro (robot description, xacro)
@@ -7,5 +7,9 @@
         <origin xyz="-0.032 0 0.0" rpy="0 0 0"/>
         <geometry>
+<<<<<<< HEAD:src/chroma_simulation/urdf/turtlebot3/robot_sensors.xacro
           <mesh filename="package://chroma_simulation/models/turtlebot3/lds.dae"
+=======
+          <mesh filename="package://cares_simulation/models/turtlebot3/lds.dae"
+>>>>>>> b0b80ff (jethexa urdf):src/cares_simulation/urdf/turtlebot3/robot_sensors.xacro
                 scale="0.001 0.001 0.001"/>
         </geometry>
