Commit message: mission planner

File: src/chroma_simulation/urdf/turtlebot3/gz_control.xacro (robot description, xacro)
@@ -11,8 +11,12 @@
         <wheel_radius>0.033</wheel_radius>
         <max_linear_acceleration>0.33</max_linear_acceleration>
+        <covariance_x>0.0001</covariance_x>
+        <covariance_y>0.0001</covariance_y>
+        <covariance_yaw>0.01</covariance_yaw>
         <topic>/model/${model_name}/cmd_vel</topic>
         <frame_id>${model_name}/odom</frame_id>
         <child_frame_id>${model_name}/base_footprint</child_frame_id>
-        <odom_topic>/model/${model_name}/odom</odom_topic>
+        <publish_odom_tf>false</publish_odom_tf>
+        <odom_topic>/model/${model_name}/odom_raw</odom_topic>
         <odom_publisher_frequency>30</odom_publisher_frequency>
         <tf_topic>/model/${model_name}/tf</tf_topic>

File: src/chroma_simulation/urdf/turtlebot3/robot_core.xacro (robot description, xacro)
@@ -17,6 +17,5 @@
         <origin xyz="-0.032 0 0.0" rpy="0 0 0"/>
         <geometry>
-          <mesh filename="package://chroma_simulation/models/turtlebot3/burger_base.dae"
-                scale="0.001 0.001 0.001"/>
+          <mesh filename="package://chroma_simulation/models/turtlebot3/burger_base.dae" scale="0.001 0.001 0.001"/>
         </geometry>
         <material name="dark"/>
@@ -47,6 +46,5 @@
           <origin xyz="0 0 0" rpy="${M_PI/2} 0 0"/>
           <geometry>
-            <mesh filename="package://chroma_simulation/models/turtlebot3/tire.dae"
-                  scale="0.001 0.001 0.001"/>
+            <mesh filename="package://chroma_simulation/models/turtlebot3/tire.dae" scale="0.001 0.001 0.001"/>
           </geometry>
           <material name="dark"/>

File: src/chroma_simulation/urdf/turtlebot3/robot_sensors.xacro (robot description, xacro)
@@ -7,6 +7,5 @@
         <origin xyz="-0.032 0 0.0" rpy="0 0 0"/>
         <geometry>
-          <mesh filename="package://chroma_simulation/models/turtlebot3/lds.dae"
-                scale="0.001 0.001 0.001"/>
+          <mesh filename="package://chroma_simulation/models/turtlebot3/lds.dae" scale="0.001 0.001 0.001"/>
         </geometry>
         <material name="dark"/>
@@ -32,5 +31,4 @@
     </joint>
     <gazebo reference="base_scan">
-      <!-- <material>Gazebo/Black</material> -->
       <sensor name="lds_sensor" type="gpu_lidar">
         <pose>0 0 0 0 0 0</pose>
@@ -48,5 +46,5 @@
           <range>
             <min>0.12</min>
-            <max>3.5</max>
+            <max>6.0</max>
           </range>
           <noise>

Commit message: rviz plugins

File: src/chroma_simulation/urdf/turtlebot3/gz_control.xacro (robot description, xacro)
@@ -11,8 +11,13 @@
         <wheel_radius>0.033</wheel_radius>
         <max_linear_acceleration>0.33</max_linear_acceleration>
+        <covariance_x>0.0001</covariance_x>
+        <covariance_y>0.0001</covariance_y>
+        <covariance_yaw>0.01</covariance_yaw>
         <topic>/model/${model_name}/cmd_vel</topic>
         <frame_id>${model_name}/odom</frame_id>
         <child_frame_id>${model_name}/base_footprint</child_frame_id>
-        <odom_topic>/model/${model_name}/odom</odom_topic>
+        <!-- <publish_odom_tf>false</publish_odom_tf> -->
+        <!-- <odom_topic>/model/${model_name}/odom_raw</odom_topic> -->
+         <odom_topic>/model/${model_name}/odom</odom_topic>
         <odom_publisher_frequency>30</odom_publisher_frequency>
         <tf_topic>/model/${model_name}/tf</tf_topic>

File: src/chroma_simulation/urdf/turtlebot3/robot_sensors.xacro (robot description, xacro)
@@ -32,5 +32,4 @@
     </joint>
     <gazebo reference="base_scan">
-      <!-- <material>Gazebo/Black</material> -->
       <sensor name="lds_sensor" type="gpu_lidar">
         <pose>0 0 0 0 0 0</pose>
@@ -48,5 +47,5 @@
           <range>
             <min>0.12</min>
-            <max>3.5</max>
+            <max>6.0</max>
           </range>
           <noise>
