Commit message: implement jethexa controller

File: src/chroma_simulation/urdf/jethexa/gz_control.xacro (robot description, xacro)
@@ -1,4 +1,8 @@
 <?xml version="1.0"?>
 <robot xmlns:xacro="http://www.ros.org/wiki/xacro">
+<<<<<<< HEAD
+=======
+  <!-- A helper macro to create an Ignition Position Controller for an articulated joint -->
+>>>>>>> d06e372 (implement jethexa controller)
   <xacro:macro name="ign_joint_controller" params="joint_name model_name">
     <plugin
@@ -18,5 +22,9 @@
   <xacro:macro name="jethexa_gz_control" params="model_name">
     <gazebo>
+<<<<<<< HEAD
       <!-- Joint State Publisher -->
+=======
+      <!-- Joint State Publisher for ALL joints -->
+>>>>>>> d06e372 (implement jethexa controller)
       <plugin
         filename="libignition-gazebo-joint-state-publisher-system.so"
@@ -24,4 +32,5 @@
         <topic>/model/${model_name}/joint_states</topic>
       </plugin>
+<<<<<<< HEAD
       <!-- ODOMETRY & TF PUBLISHER -->
       <plugin
@@ -36,4 +45,6 @@
         <dimensions>2</dimensions>
       </plugin>
+=======
+>>>>>>> d06e372 (implement jethexa controller)
       <!-- Head Controllers -->
       <xacro:ign_joint_controller joint_name="head_pan_joint" model_name="${model_name}"/>

File: src/chroma_simulation/urdf/jethexa/robot_sensors.xacro (robot description, xacro)
@@ -46,5 +46,9 @@
         </lidar>
         <topic>/model/${model_name}/scan</topic>
+<<<<<<< HEAD
         <gz_frame_id>${model_name}/lidar_visual_link</gz_frame_id>
+=======
+        <gz_frame_id>lidar_visual_link</gz_frame_id>
+>>>>>>> d06e372 (implement jethexa controller)
       </sensor>
     </gazebo>
@@ -63,5 +67,9 @@
         <update_rate>200</update_rate>
         <topic>/model/${model_name}/imu</topic>
+<<<<<<< HEAD
         <gz_frame_id>${model_name}/imu_link</gz_frame_id>
+=======
+        <gz_frame_id>imu_link</gz_frame_id>
+>>>>>>> d06e372 (implement jethexa controller)
       </sensor>
     </gazebo>
@@ -112,5 +120,9 @@
         </camera>
         <topic>/model/${model_name}/camera</topic>
+<<<<<<< HEAD
         <gz_frame_id>${model_name}/camera_color_optical_frame</gz_frame_id>
+=======
+        <gz_frame_id>camera_color_optical_frame</gz_frame_id>
+>>>>>>> d06e372 (implement jethexa controller)
       </sensor>
     </gazebo>

File: src/chroma_simulation/urdf/turtlebot3/robot_core.xacro (robot description, xacro)
@@ -17,4 +17,5 @@
         <origin xyz="-0.032 0 0.0" rpy="0 0 0"/>
         <geometry>
+<<<<<<< HEAD
 <<<<<<< HEAD:src/chroma_simulation/urdf/turtlebot3/robot_core.xacro
           <mesh filename="package://chroma_simulation/models/turtlebot3/burger_base.dae"
@@ -22,4 +23,7 @@
           <mesh filename="package://cares_simulation/models/turtlebot3/burger_base.dae"
 >>>>>>> b0b80ff (jethexa urdf):src/cares_simulation/urdf/turtlebot3/robot_core.xacro
+=======
+          <mesh filename="package://chroma_simulation/models/turtlebot3/burger_base.dae"
+>>>>>>> d06e372 (implement jethexa controller)
                 scale="0.001 0.001 0.001"/>
         </geometry>
@@ -51,4 +55,5 @@
           <origin xyz="0 0 0" rpy="${M_PI/2} 0 0"/>
           <geometry>
+<<<<<<< HEAD
 <<<<<<< HEAD:src/chroma_simulation/urdf/turtlebot3/robot_core.xacro
             <mesh filename="package://chroma_simulation/models/turtlebot3/tire.dae"
@@ -56,4 +61,7 @@
             <mesh filename="package://cares_simulation/models/turtlebot3/tire.dae"
 >>>>>>> b0b80ff (jethexa urdf):src/cares_simulation/urdf/turtlebot3/robot_core.xacro
+=======
+            <mesh filename="package://chroma_simulation/models/turtlebot3/tire.dae"
+>>>>>>> d06e372 (implement jethexa controller)
                   scale="0.001 0.001 0.001"/>
           </geometry>

File: src/chroma_simulation/urdf/turtlebot3/robot_sensors.xacro (robot description, xacro)
@@ -7,4 +7,5 @@
         <origin xyz="-0.032 0 0.0" rpy="0 0 0"/>
         <geometry>
+<<<<<<< HEAD
 <<<<<<< HEAD:src/chroma_simulation/urdf/turtlebot3/robot_sensors.xacro
           <mesh filename="package://chroma_simulation/models/turtlebot3/lds.dae"
@@ -12,4 +13,7 @@
           <mesh filename="package://cares_simulation/models/turtlebot3/lds.dae"
 >>>>>>> b0b80ff (jethexa urdf):src/cares_simulation/urdf/turtlebot3/robot_sensors.xacro
+=======
+          <mesh filename="package://chroma_simulation/models/turtlebot3/lds.dae"
+>>>>>>> d06e372 (implement jethexa controller)
                 scale="0.001 0.001 0.001"/>
         </geometry>
